Commit message: fixed steer joints on rear wheels

File: steerbot/urdf/steerbot.xacro (robot description, xacro)
@@ -279,5 +279,5 @@
         <dynamics damping="${bearing_damping}" friction="${bearing_friction}"/>
     </joint>
-    <joint name="rear_left_steer_bearing" type="continuous">
+    <joint name="rear_left_steer_bearing" type="fixed">
         <!--
             The wheel_rad/3.0 gives some space between strut and chassis that
@@ -300,5 +300,5 @@
         <dynamics damping="${bearing_damping}" friction="${bearing_friction}"/>
     </joint>
-    <joint name="rear_right_steer_bearing" type="continuous">
+    <joint name="rear_right_steer_bearing" type="fixed">
         <!--
             The wheel_rad/3.0 gives some space between strut and chassis that
